File: key1/key1.kicad_pcb (KiCad board)
At the start: 2 copper layers, 43.8 x 106.2 mm, 9 parts

Commit message: back
Parts:
- added G***: LOGO, lib:goldbug.cpvBcu, B.Cu at (182.8, 71.5)
- added G***: LOGO, lib:goldbug.cpv, B.Cu at (182.8, 71.5)

Commit message: p
Parts:
- added G***: LOGO, lib:patent, B.Cu at (183.1, 145.2)
