File: key2/key2.kicad_pcb (KiCad board)
At the start: 2 copper layers, 42.6 x 108.2 mm, 9 parts

Commit message: update
Routing:
- added copper zone on B.Cu, net (none)
- added copper zone on F.Cu, net (none)
Changed lines of the file:
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@@
   (gr_line (start 126.24 104.18) (end 117.07 104.11) (angle 90) (layer Edge.Cuts) (width 0.15))
   (gr_line (start 128.4 106.27) (end 126.24 104.18) (angle 90) (layer Edge.Cuts) (width 0.15))
+  (zone (net 0) (net_name "") (layer F.Cu) (hatch edge 0.508)
+    (connect_pads (clearance 0.508))
+    (min_thickness 0.254)
+    (fill (arc_segments 16) (thermal_gap 0.508) (thermal_bridge_width 0.508))
+    (polygon
+      (pts
+        (xy 100.5 57.5) (xy 166.5 57.25) (xy 154.75 183) (xy 106.75 182.5) (xy 100.25 57)
+      )
+    )
+  )
+  (zone (net 0) (net_name "") (layer B.Cu) (hatch edge 0.508)
+    (connect_pads (clearance 0.508))
+    (min_thickness 0.254)
+    (fill (arc_segments 16) (thermal_gap 0.508) (thermal_bridge_width 0.508))
+    (polygon
+      (pts
+        (xy 100.5 57.5) (xy 166.25 57.5) (xy 154.5 183) (xy 107 182.25) (xy 100.5 57.5)
+      )
+    )
+  )
 )

Commit message: back
Parts:
- added G***: LOGO, lib:goldbug.cpvBcu, B.Cu at (132.5, 89.2)
- added G***: LOGO, lib:goldbug.cpv, B.Cu at (132.5, 89.2)
- moved G*** 0.06 mm to (132.4, 88.0)

Commit message: p
Parts:
- added G***: LOGO, lib:patent, B.Cu at (132.6, 164.7)
