File: key3/key3.kicad_pcb (KiCad board)
At the start: 2 copper layers, 31.5 x 107.1 mm, 11 parts

Commit message: back
Parts:
- added G***: LOGO, lib:goldbug.cpv, B.Cu at (180.5, 72.9)
- added G***: LOGO, lib:goldbug.cpvBcu, B.Cu at (180.5, 72.9)

Commit message: p
Parts:
- added G***: LOGO, lib:patent, B.Cu at (180.5, 142.8)
