File: key4/key4.kicad_pcb (KiCad board)
At the start: 2 copper layers, 41.2 x 107.7 mm, 9 parts

Commit message: back
Parts:
- added G***: LOGO, lib:goldbug.cpv, B.Cu at (130.0, 60.8)
- added G***: LOGO, lib:goldbug.cpvBcu, B.Cu at (130.0, 60.8)

Commit message: p
Parts:
- added G***: LOGO, lib:patent, B.Cu at (130.0, 137.8)
