File: key5/key5.kicad_pcb (KiCad board)
At the start: 2 copper layers, 40.8 x 110.8 mm, 9 parts

Commit message: back
Parts:
- added G***: LOGO, lib:goldbug.cpvBcu, B.Cu at (163.4, 65.0)
- added G***: LOGO, lib:goldbug.cpv, B.Cu at (163.4, 65.0)

Commit message: p
Parts:
- added G***: LOGO, lib:patent, B.Cu at (163.2, 135.1)
